Commit message: Added ground calibration

File: ackermann_vehicle_description/urdf/em_3905_camera.urdf.xacro (robot description, xacro)
@@ -383,9 +383,9 @@
     cam_info_topic="camera/camera_info"
     update_rate="30"
-    res_x="640"
-    res_y="480"
+    res_x="1280"
+    res_y="720"
     image_format="R8G8B8"
     hfov="90">
-    <origin xyz="0.305 0 0.11" rpy="0 0 0" />
+    <origin xyz="0.305 0 0.3" rpy="0 0 0" />
   </xacro:generic_camera>
   <gazebo>
